Commit message: fix: robust JSON parser for Nemotron, honest AI/fallback HUD reporting, REP-103 serial URDF structure, and accurate documentation

File: Exports/kinetic_claw_145mm.urdf (robot description, URDF)
Before this commit: robot kinetic_claw_145mm, 4 links, 3 joints
Links:
- added link turret_link, mass 0.0100
- link base_link: geometry collision cylinder length=0.06000 radius=0.04000; visual cylinder length=0.06000 radius=0.04000
- link distal_jaw_link: geometry collision box size=0.02200 0.17135 0.02200; visual box size=0.02200 0.17135 0.02200
- link proximal_link: geometry collision box size=0.02600 0.20860 0.02600; visual box size=0.02600 0.20860 0.02600
Joints:
- added joint ee_fixed_joint: type fixed, parent distal_jaw_link, child ee_tip, origin xyz=0.00000 -0.17135 0.00000 rpy=0 0 0
- joint base_yaw_joint: axis 0.0000 1.0000 0.0000 -> 0.0000 0.0000 -1.0000; child proximal_link -> turret_link; origin xyz=0.0000 0.0600 0.0000 rpy=0 0 0 -> xyz=0.00000 0.00000 0.06000 rpy=0 0 0
- joint elbow_pitch_joint: axis 0.0000 0.0000 1.0000 -> -1.0000 0.0000 0.0000; child ee_tip -> distal_jaw_link; origin xyz=0.2086 0.0000 0.0000 rpy=0 0 0 -> xyz=0.00000 -0.20860 0.00000 rpy=0 0 0; parent distal_jaw_link -> proximal_link
- joint shoulder_pitch_joint: axis 0.0000 0.0000 1.0000 -> -1.0000 0.0000 0.0000; child distal_jaw_link -> proximal_link; origin xyz=0.0000 0.0000 0.0000 rpy=0 0 0 -> xyz=0.00000 0.00000 0.00000 rpy=0 0 0; parent proximal_link -> turret_link

File: Exports/kinetic_claw_70mm.urdf (robot description, URDF)
Before this commit: robot kinetic_claw_70mm, 4 links, 3 joints
Links:
- added link turret_link, mass 0.0100
- link base_link: geometry collision cylinder length=0.06000 radius=0.04000; visual cylinder length=0.06000 radius=0.04000
- link distal_jaw_link: geometry collision box size=0.02200 0.08510 0.02200; visual box size=0.02200 0.08510 0.02200
- link proximal_link: geometry collision box size=0.02600 0.10360 0.02600; visual box size=0.02600 0.10360 0.02600
Joints:
- added joint ee_fixed_joint: type fixed, parent distal_jaw_link, child ee_tip, origin xyz=0.00000 -0.08510 0.00000 rpy=0 0 0
- joint base_yaw_joint: axis 0.0000 1.0000 0.0000 -> 0.0000 0.0000 -1.0000; child proximal_link -> turret_link; origin xyz=0.0000 0.0600 0.0000 rpy=0 0 0 -> xyz=0.00000 0.00000 0.06000 rpy=0 0 0
- joint elbow_pitch_joint: axis 0.0000 0.0000 1.0000 -> -1.0000 0.0000 0.0000; child ee_tip -> distal_jaw_link; origin xyz=0.1036 0.0000 0.0000 rpy=0 0 0 -> xyz=0.00000 -0.10360 0.00000 rpy=0 0 0; parent distal_jaw_link -> proximal_link
- joint shoulder_pitch_joint: axis 0.0000 0.0000 1.0000 -> -1.0000 0.0000 0.0000; child distal_jaw_link -> proximal_link; origin xyz=0.0000 0.0000 0.0000 rpy=0 0 0 -> xyz=0.00000 0.00000 0.00000 rpy=0 0 0; parent proximal_link -> turret_link
